File: hardware/Make files/Active/_autosave-CAN_Firewall.kicad_pcb (KiCad board)
At the start: 2 copper layers, 68 x 44 mm, 60 parts, among them CON1 BARREL_JACK, CON2 AVR-JTAG-10, CON3 AVR-AW-6, J1 +5V_SRC, J2 DB9, J3 DB9, P1 USB_OTG, P2 USB_OTG, P3 DIAG Port, SW1 SPST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

Commit message: V1.11 Schematic and PCB layout
Routing:
- net GND: track 303.8 -> 333.1 mm, vias 59 -> 65
Changed lines of the file:
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@@
   (general
     (links 193)
-    (no_connects 1)
+    (no_connects 0)
     (area 39.949999 110.949999 108.050001 155.050001)
     (thickness 1.6)
-    (drawings 44)
-    (tracks 1308)
+    (drawings 43)
+    (tracks 1332)
     (zones 0)
     (modules 60)
@@
     (pad 3 thru_hole circle (at 4.8 -10.75 180) (size 3.75 3.75) (drill 3.05) (layers *.Cu *.Mask F.SilkS))
   )
-  (dimension 6.8 (width 0.3) (layer Cmts.User)
-    (gr_text "6.800 mm" (at 101 159.25) (layer Cmts.User)
-      (effects (font (size 1.5 1.5) (thickness 0.3)))
-    )
-    (feature1 (pts (xy 97.6 151.9) (xy 97.6 160.6)))
-    (feature2 (pts (xy 104.4 151.9) (xy 104.4 160.6)))
-    (crossbar (pts (xy 104.4 157.9) (xy 97.6 157.9)))
-    (arrow1a (pts (xy 97.6 157.9) (xy 98.726504 157.313579)))
-    (arrow1b (pts (xy 97.6 157.9) (xy 98.726504 158.486421)))
-    (arrow2a (pts (xy 104.4 157.9) (xy 103.273496 157.313579)))
-    (arrow2b (pts (xy 104.4 157.9) (xy 103.273496 158.486421)))
-  )
   (gr_text PWR (at 75.5 112.1) (layer F.SilkS)
     (effects (font (size 1.5 1.5) (thickness 0.3)))
@@
   (segment (start 47.3 117.7) (end 47.3 118.2) (width 0.25) (layer F.Cu) (net 1))
   (segment (start 48.3009 116.6991) (end 47.3 117.7) (width 0.25) (layer F.Cu) (net 1))
+  (segment (start 75.2 133.7) (end 75.2 132.5) (width 0.25) (layer B.Cu) (net 2))
+  (segment (start 73.2 130.9) (end 72.7 130.9) (width 0.25) (layer F.Cu) (net 2))
+  (segment (start 73.4 130.7) (end 73.2 130.9) (width 0.25) (layer F.Cu) (net 2))
+  (via (at 73.4 130.7) (size 0.6) (drill 0.4) (layers F.Cu B.Cu) (net 2))
+  (segment (start 75.2 132.5) (end 73.4 130.7) (width 0.25) (layer B.Cu) (net 2))
+  (segment (start 51.6 134.8) (end 53.7 134.8) (width 0.25) (layer B.Cu) (net 2))
+  (segment (start 51.9 141.5) (end 52.2 141.2) (width 0.25) (layer B.Cu) (net 2))
+  (via (at 51.9 141.5) (size 0.6) (drill 0.4) (layers F.Cu B.Cu) (net 2))
+  (segment (start 51.9 138.6) (end 51.9 141.5) (width 0.25) (layer F.Cu) (net 2))
+  (segment (start 54.7 135.8) (end 51.9 138.6) (width 0.25) (layer F.Cu) (net 2))
+  (via (at 54.7 135.8) (size 0.6) (drill 0.4) (layers F.Cu B.Cu) (net 2))
+  (segment (start 53.7 134.8) (end 54.7 135.8) (width 0.25) (layer B.Cu) (net 2))
+  (segment (start 101.6 141.2) (end 100.4 142.4) (width 0.25) (layer B.Cu) (net 2))
+  (segment (start 101.8 153.4) (end 102.2 153.4) (width 0.25) (layer F.Cu) (net 2))
+  (segment (start 101.3 152.9) (end 101.8 153.4) (width 0.25) (layer F.Cu) (net 2))
+  (via (at 101.3 152.9) (size 0.6) (drill 0.4) (layers F.Cu B.Cu) (net 2))
+  (segment (start 101.3 149.9) (end 101.3 152.9) (width 0.25) (layer B.Cu) (net 2))
+  (segment (start 101.5 149.7) (end 101.3 149.9) (width 0.25) (layer B.Cu) (net 2))
+  (via (at 101.5 149.7) (size 0.6) (drill 0.4) (layers F.Cu B.Cu) (net 2))
+  (segment (start 101.5 144.7) (end 101.5 149.7) (width 0.25) (layer F.Cu) (net 2))
+  (segment (start 100.6 143.8) (end 101.5 144.7) (width 0.25) (layer F.Cu) (net 2))
+  (segment (start 100.4 143.8) (end 100.6 143.8) (width 0.25) (layer F.Cu) (net 2))
+  (via (at 100.4 143.8) (size 0.6) (drill 0.4) (layers F.Cu B.Cu) (net 2))
+  (segment (start 100.4 142.4) (end 100.4 143.8) (width 0.25) (layer B.Cu) (net 2))
   (segment (start 88.4 129) (end 90 129) (width 0.25) (layer F.Cu) (net 2))
   (segment (start 90.1 129.1) (end 90.2 129.1) (width 0.25) (layer B.Cu) (net 2))
@@
   (segment (start 102.909 138.309) (end 102.2 137.6) (width 0.5) (layer F.Cu) (net 5))
   (segment (start 42.3 138.069) (end 42.54 138.309) (width 0.5) (layer B.Cu) (net 5))
+  (segment (start 90.2 120.5) (end 89.5 121.2) (width 0.25) (layer F.Cu) (net 6))
+  (segment (start 83 128.2) (end 83 130.1) (width 0.25) (layer F.Cu) (net 6))
+  (segment (start 83.8 127.4) (end 83 128.2) (width 0.25) (layer F.Cu) (net 6))
+  (segment (start 87.4 127.4) (end 83.8 127.4) (width 0.25) (layer F.Cu) (net 6))
+  (segment (start 89.5 125.3) (end 87.4 127.4) (width 0.25) (layer F.Cu) (net 6))
+  (segment (start 89.5 121.2) (end 89.5 125.3) (width 0.25) (layer F.Cu) (net 6))
+  (segment (start 77.4 128.2) (end 77.1 128.2) (width 0.25) (layer B.Cu) (net 6))
+  (segment (start 77.1 128.2) (end 76.9 128.4) (width 0.25) (layer B.Cu) (net 6))
   (segment (start 94.225 132.6) (end 94.2 132.575) (width 0.25) (layer F.Cu) (net 6))
   (segment (start 94.2 132.575) (end 94.2 131) (width 0.25) (layer F.Cu) (net 6))
@@
   (segment (start 95.4 121.5) (end 97.475 123.575) (width 0.25) (layer F.Cu) (net 6))
   (segment (start 97.475 123.575) (end 97.475 125.4) (width 0.25) (layer F.Cu) (net 6))
-  (segment (start 83 129.5) (end 83 130.1) (width 0.25) (layer F.Cu) (net 6))
   (segment (start 93.6 131) (end 94.2 131) (width 0.5) (layer F.Cu) (net 6))
   (segment (start 94.2 131) (end 94.8 131) (width 0.5) (layer F.Cu) (net 6))
   (segment (start 83.4 130.1) (end 86.5 130.1) (width 0.5) (layer F.Cu) (net 6))
+  (segment (start 86.5 130.1) (end 88.4 132) (width 0.5) (layer F.Cu) (net 6))
+  (segment (start 83 130.1) (end 83.4 130.1) (width 0.5) (layer F.Cu) (net 6))
   (via (at 77.4 128.2) (size 0.75) (drill 0.5) (layers F.Cu B.Cu) (net 6))
+  (segment (start 80.3 130.1) (end 83 130.1) (width 0.5) (layer F.Cu) (net 6))
+  (segment (start 78.4 128.2) (end 80.3 130.1) (width 0.5) (layer F.Cu) (net 6))
   (segment (start 77.4 128.2) (end 78.4 128.2) (width 0.5) (layer F.Cu) (net 6))
-  (segment (start 78.4 128.2) (end 80.3 130.1) (width 0.5) (layer F.Cu) (net 6))
-  (segment (start 80.3 130.1) (end 83.4 130.1) (width 0.5) (layer F.Cu) (net 6))
   (via (at 72 128.4) (size 0.6) (drill 0.4) (layers F.Cu B.Cu) (net 6))
+  (segment (start 76 128.4) (end 76.9 128.4) (width 0.5) (layer B.Cu) (net 6))
   (segment (start 72 128.4) (end 76 128.4) (width 0.5) (layer B.Cu) (net 6))
-  (segment (start 76 128.4) (end 76.9 128.4) (width 0.5) (layer B.Cu) (net 6))
   (segment (start 76.9 128.4) (end 77.2 128.4) (width 0.5) (layer B.Cu) (net 6))
-  (segment (start 86.5 130.1) (end 88.4 132) (width 0.5) (layer F.Cu) (net 6))
   (segment (start 59.3 128.1) (end 59.3 130.8) (width 0.5) (layer F.Cu) (net 6))
   (segment (start 56.6 133.5) (end 54.4 133.5) (width 0.5) (layer F.Cu) (net 6))
@@
   (segment (start 49.9 137.275) (end 50.625 137.275) (width 0.25) (layer F.Cu) (net 6))
   (segment (start 50.625 137.275) (end 54.4 133.5) (width 0.25) (layer F.Cu) (net 6))
-  (segment (start 83 130.1) (end 82.9 130.1) (width 0.25) (layer F.Cu) (net 6))
   (segment (start 83.6 141.5) (end 84.5 142.4) (width 0.25) (layer F.Cu) (net 6))
   (segment (start 89.5 137) (end 88.5 136) (width 0.25) (layer F.Cu) (net 6))
@@
   (segment (start 86.7 142.4) (end 87.7 141.4) (width 0.25) (layer F.Cu) (net 6))
   (segment (start 84.5 142.4) (end 86.7 142.4) (width 0.25) (layer F.Cu) (net 6))
-  (segment (start 88.1 126.8) (end 87.5 127.4) (width 0.25) (layer F.Cu) (net 6))
   (segment (start 93.5 120.5) (end 90.2 120.5) (width 0.25) (layer F.Cu) (net 6))
-  (segment (start 90.2 120.5) (end 89.5 121.2) (width 0.25) (layer F.Cu) (net 6))
-  (segment (start 89.5 121.2) (end 89.5 125.4) (width 0.25) (layer F.Cu) (net 6))
-  (segment (start 89.5 125.4) (end 88.1 126.8) (width 0.25) (layer F.Cu) (net 6))
   (segment (start 94.4 121.4) (end 93.5 120.5) (width 0.25) (layer F.Cu) (net 6))
-  (segment (start 83 128.2) (end 83 129.5) (width 0.25) (layer F.Cu) (net 6))
-  (segment (start 83.8 127.4) (end 83 128.2) (width 0.25) (layer F.Cu) (net 6))
-  (segment (start 87.5 127.4) (end 83.8 127.4) (width 0.25) (layer F.Cu) (net 6))
   (segment (start 96.7 122.8) (end 95.4 121.5) (width 0.25) (layer F.Cu) (net 6))
   (segment (start 97.475 123.575) (end 96.7 122.8) (width 0.25) (layer F.Cu) (net 6))
